Commit message: camera

File: robot/urdf/myfirst.urdf (robot description, URDF)
Before this commit: robot myfirst, 6 links, 5 joints
Links:
- added link camera_link, mass 0.1; visual box size=0.5 0.5 0.5
Joints:
- added joint fix_3: type fixed, parent link_4, child camera_link, origin xyz=0 0 2 rpy=0 0 0 

Commit message: new launch file , new camera saver script, new video and photo folder

File: robot/urdf/myfirst.urdf (robot description, URDF)
Before this commit: robot myfirst, 7 links, 6 joints
Joints:
- joint fix_3: origin xyz=0 0 2 rpy=0 0 0  -> xyz=5.25 0 1.25 rpy=0 0 0 
